File: SEPIC.kicad_pcb (KiCad board)
At the start: 2 copper layers, 106.5 x 67.1 mm, 30 parts, among them J1 Screw_Terminal_01x02, J3 Screw_Terminal_01x02, J4 Conn_01x04_Male, J5 Conn_01x02_Male, J6 Conn_01x03_Male, J7 Screw_Terminal_01x02, U1 AP2205, U2 XL6009, U3 MCP48FVB21

Commit message: Added license related text
Other:
- board text added: "SPI SEPIC v0.1 License: CC-BY-SA 4.0"
- board text removed: "SPI SEPIC v0.1 License: CC BY 4.0"
